Commit message: objects 3x larger

File: resources/models/environment_assets/objects/cube.urdf (robot description, URDF)
Before this commit: robot box, 1 links, 0 joints
Links:
- link base_link: geometry collision box size=3.0 3.0 3.0; visual box size=3.0 3.0 3.0

File: resources/models/environment_assets/objects/cuboidal_rod.urdf (robot description, URDF)
Before this commit: robot box, 1 links, 0 joints
Links:
- link base_link: geometry collision box size=0.45 0.45 9.0; visual box size=0.45 0.45 3.0

File: resources/models/environment_assets/objects/small_cube.urdf (robot description, URDF)
Before this commit: robot box, 1 links, 0 joints
Links:
- link base_link: geometry collision box size=1.2 1.2 1.2; visual box size=1.2 1.2 1.2

File: resources/models/environment_assets/objects/small_sphere.urdf (robot description, URDF)
Before this commit: robot sphere, 1 links, 0 joints
Links:
- link base_link: geometry collision sphere radius=0.9; visual sphere radius=0.9

File: resources/models/environment_assets/objects/sphere.urdf (robot description, URDF)
Before this commit: robot sphere, 1 links, 0 joints
Links:
- link base_link: geometry collision sphere radius=1.5; visual sphere radius=1.5
